Commit message: Vision Line connected to ROS-GZ

File: morpho_gnn_robot/install/morpho_robot/share/morpho_robot/urdf/anymal.urdf (robot description, URDF)
Before this commit: robot anymal, 22 links, 21 joints
Links:
- added link camera_link, mass 0.1; visual box size=0.05 0.05 0.05
Joints:
- added joint camera_joint: type fixed, parent base, child camera_link, origin xyz=0.3 0 0.1 rpy=0 0 0
